File: biscotti/biscotti.kicad_pcb (KiCad board)
At the start: 2 copper layers, 60 x 20 mm, 38 parts, among them J1 Conn_02x01, J2 Conn_02x06_Odd_Even, J3 Conn_01x01, J4 RJ45_Halo_HFJ11-x2450E-LxxRL, U1 LAN8720A

Commit message: wip
Parts:
- moved C13 103.2 mm to (128.2, 97.7), turned to 90 degrees
- moved C14 101.1 mm to (131.1, 97.7), turned to 90 degrees
- moved C1 0.50 mm to (152.7, 99.0)
- moved C12 0.50 mm to (168.8, 99.0)
- moved FB1 0.50 mm to (163.3, 99.0)
- moved J3 0.50 mm to (142.8, 98.8)
- moved R10 0.50 mm to (147.2, 99.0)
- moved R11 0.50 mm to (157.9, 99.0)
Routing:
- net GND: track 40.7 -> 108.2 mm
- net EGND: track 0.00 -> 44.9 mm
- net VDDA: track 28.7 -> 57.4 mm, vias 0 -> 1
- net VDD: track 19.1 -> 32.0 mm
- net /nINT: track 20.6 -> 18.7 mm
Other:
- board size 60 x 20 mm -> 69.2 x 20 mm

Commit message: biscotti 1.0 and 1.1
Parts:
- moved R1 107.1 mm to (137.4, 82.8), turned to 180 degrees
- moved C8 100.1 mm to (134.0, 97.7), turned to 90 degrees
- moved C2 99.3 mm to (142.7, 82.8), turned to 180 degrees
- moved C6 96.5 mm to (136.8, 97.7), turned to 90 degrees
- moved C3 96.3 mm to (148.2, 82.8)
- moved R17 87.3 mm to (157.0, 84.3), turned to 90 degrees
- moved R18 78.0 mm to (167.8, 83.0)
- moved C10 68.4 mm to (163.4, 96.5), turned to 180 degrees
- moved C11 66.5 mm to (168.8, 96.5)
- moved J1 14.6 mm to (133.0, 83.0), turned to 180 degrees
- moved R13 4.32 mm to (162.2, 83.0), turned to 0 degrees
- moved R6 0.75 mm to (147.5, 87.0)
- moved R8 0.75 mm to (150.2, 87.0)
- moved R2 0.31 mm to (142.2, 88.6)
- moved R3 0.31 mm to (142.2, 85.8)
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Routing:
- net VDD: track 32.0 -> 92.3 mm, vias 2 -> 5
- net /LED1: track 0.00 -> 42.9 mm, vias 0 -> 2
- net GND: track 108.2 -> 150.2 mm, vias 0 -> 6
- net VDDA: track 57.4 -> 96.5 mm, vias 1 -> 4
- net /G-: track 0.00 -> 33.9 mm
- net /MDC: track 0.00 -> 28.9 mm, vias 0 -> 1
- net /MDIO: track 0.00 -> 27.4 mm, vias 0 -> 1
- net /Y-: track 0.00 -> 23.1 mm
- net EGND: track 44.9 -> 22.7 mm, vias 0 -> 2
- net /VDDCR: track 0.00 -> 12.9 mm, vias 0 -> 2
- net Net-(U1-RBIAS): track 4.30 -> 7.47 mm
- net /nRST: track 13.2 -> 10.4 mm
- net /Clk: track 37.9 -> 35.3 mm
- net /LED2: track 0.00 -> 2.46 mm
- net /TXD[1]: track 39.4 -> 41.4 mm
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- added copper zone on B.Cu, net EGND
- added copper zone on F.Cu, net EGND
- added copper zone on B.Cu, net GND
- added copper zone on F.Cu, net GND
Other:
- board size 69.2 x 20 mm -> 74.8 x 20 mm
- board text added: "Biscotti v1.1"
- board text added: "CLK"
- board text added: "GND"
- board text added: "RXD0"
- board text added: "RXD1"
- board text added: "RXERR"
- board text added: "RXV"
- board text added: "TXD0"
- board text added: "TXD1"
- board text added: "TXV"
